File: Rev_A/Raspberry_Pi_Pico_Keyboard.kicad_sch (KiCad schematic)
At the start: 9 parts, among them J1 Conn_01x20_Pin, J2 Conn_01x20_Pin

Commit message: Fix title typo in Raspberry Pi Pico Keyboard schematic
Other:
- title: Raspberry_Pi_Picp_Keyboard -> Raspberry_Pi_Pico_Keyboard
Changed lines of the file:
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@@
 	(paper "A4")
 	(title_block
-		(title "Raspberry_Pi_Picp_Keyboard")
+		(title "Raspberry_Pi_Pico_Keyboard")
 		(date "2026-08-25")
 		(rev "Rev. A")
